File: Protopico/Protopico.kicad_sch (KiCad schematic)
At the start: 56 parts, among them J1 Conn_01x03, J10 Conn_02x02_Odd_Even, J12 Conn_01x03, J13 USB_C_Receptacle, J2 Conn_01x01, J3 Conn_01x01, J4 Conn_01x01, J5 Conn_02x13_Odd_Even, J6 Conn_01x02, J7 Conn_02x02_Odd_Even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

Commit message: improved pcb and schematic
Parts:
- added C19: 100nF, Capacitor_SMD:C_1206_3216Metric_Pad1.33x1.80mm_HandSolder, symbol Device:C
- added U5: SRV05-4, Package_TO_SOT_SMD:SOT-23-6, symbol Power_Protection:SRV05-4
- J13: value USB_C_Receptacle -> USB_C 2.0
Connections:
- net +3V3: now also C19.1
- net GND: now also C19.2, U5.2 (VN)
- net USB_D+: now also U5.3 (IO2)
- net USB_D-: now also U5.1 (IO1)
- net VBUS: now also U5.5 (VP)
Other:
- moved on the sheet: C1, C2, D3, R1, R13, R9, SW1, U1

Commit message: improved pcb
Parts:
- removed U5: SRV05-4, Package_TO_SOT_SMD:SOT-23-6, symbol Power_Protection:SRV05-4
Changed lines of the file:
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@@
   (junction (at 213.36 41.91) (diameter 0) (color 0 0 0 0)
   )
-  (junction (at 59.69 35.56) (diameter 0) (color 0 0 0 0)
-  )
   (junction (at 55.88 104.14) (diameter 0) (color 0 0 0 0)
   )
@@
   (junction (at 121.92 157.48) (diameter 0) (color 0 0 0 0)
   )
-  (junction (at 48.26 40.64) (diameter 0) (color 0 0 0 0)
-  )
   (junction (at 229.87 44.45) (diameter 0) (color 0 0 0 0)
   )
@@
   (junction (at 247.65 20.32) (diameter 0) (color 0 0 0 0)
   )
-  (junction (at 63.5 74.93) (diameter 0) (color 0 0 0 0)
-  )
   (junction (at 157.48 92.71) (diameter 0) (color 0 0 0 0)
   )
@@
     (stroke (width 0) (type default) (color 0 0 0 0))
   )
-  (wire (pts (xy 59.69 44.45) (xy 59.69 35.56))
-    (stroke (width 0) (type default) (color 0 0 0 0))
-  )
   (wire (pts (xy 45.72 162.56) (xy 45.72 163.83))
     (stroke (width 0) (type default) (color 0 0 0 0))
@@
     (stroke (width 0) (type default) (color 0 0 0 0))
   )
-  (wire (pts (xy 48.26 60.96) (xy 48.26 40.64))
-    (stroke (width 0) (type default) (color 0 0 0 0))
-  )
-  (wire (pts (xy 63.5 71.12) (xy 63.5 74.93))
-    (stroke (width 0) (type default) (color 0 0 0 0))
-  )
   (wire (pts (xy 149.86 22.86) (xy 167.64 22.86))
     (stroke (width 0) (type default) (color 0 0 0 0))
@@
     (stroke (width 0) (type default) (color 0 0 0 0))
   )
-  (wire (pts (xy 63.5 74.93) (xy 52.07 74.93))
-    (stroke (width 0) (type default) (color 0 0 0 0))
-  )
   (wire (pts (xy 68.58 93.98) (xy 68.58 96.52))
     (stroke (width 0) (type default) (color 0 0 0 0))
@@
     (stroke (width 0) (type default) (color 0 0 0 0))
   )
-  (wire (pts (xy 43.18 35.56) (xy 59.69 35.56))
+  (wire (pts (xy 43.18 35.56) (xy 88.9 35.56))
     (stroke (width 0) (type default) (color 0 0 0 0))
   )
@@
     (stroke (width 0) (type default) (color 0 0 0 0))
   )
-  (wire (pts (xy 48.26 40.64) (xy 58.42 40.64))
-    (stroke (width 0) (type default) (color 0 0 0 0))
-  )
-  (wire (pts (xy 50.8 44.45) (xy 59.69 44.45))
-    (stroke (width 0) (type default) (color 0 0 0 0))
-  )
   (polyline (pts (xy 106.68 76.2) (xy 106.68 124.46))
     (stroke (width 0) (type default) (color 0 0 0 0))
@@
     (stroke (width 0) (type default) (color 0 0 0 0))
   )
-  (wire (pts (xy 96.52 74.93) (xy 63.5 74.93))
+  (wire (pts (xy 52.07 74.93) (xy 96.52 74.93))
     (stroke (width 0) (type default) (color 0 0 0 0))
   )
@@
     (stroke (width 0) (type default) (color 0 0 0 0))
   )
-  (wire (pts (xy 59.69 35.56) (xy 88.9 35.56))
-    (stroke (width 0) (type default) (color 0 0 0 0))
-  )
   (wire (pts (xy 40.64 43.18) (xy 43.18 43.18))
     (stroke (width 0) (type default) (color 0 0 0 0))
@@
     (stroke (width 0) (type default) (color 0 0 0 0))
   )
-  (wire (pts (xy 43.18 40.64) (xy 48.26 40.64))
+  (wire (pts (xy 43.18 40.64) (xy 58.42 40.64))
     (stroke (width 0) (type default) (color 0 0 0 0))
   )
@@
     (stroke (width 0) (type default) (color 0 0 0 0))
   )
-  (wire (pts (xy 50.8 55.88) (xy 50.8 44.45))
-    (stroke (width 0) (type default) (color 0 0 0 0))
-  )
   (wire (pts (xy 114.3 125.73) (xy 127 125.73))
     (stroke (width 0) (type default) (color 0 0 0 0))
@@
     (stroke (width 0) (type default) (color 0 0 0 0))
   )
-  (wire (pts (xy 50.8 60.96) (xy 48.26 60.96))
-    (stroke (width 0) (type default) (color 0 0 0 0))
-  )
   (wire (pts (xy 40.64 35.56) (xy 43.18 35.56))
     (stroke (width 0) (type default) (color 0 0 0 0))
@@
     (pin "1")
   )
-  (symbol (lib_id "power:VBUS") (at 63.5 45.72 0) (unit 1)
-    (in_bom yes) (on_board yes) (fields_autoplaced)
-    (property "Reference" "#PWR0135" (id 0) (at 63.5 49.53 0)
-      (effects (font (size 1.27 1.27)) hide)
-    )
-    (property "Value" "VBUS" (id 1) (at 63.5 40.64 0))
-    (property "Footprint" "" (id 2) (at 63.5 45.72 0)
-      (effects (font (size 1.27 1.27)) hide)
-    )
-    (property "Datasheet" "" (id 3) (at 63.5 45.72 0)
-      (effects (font (size 1.27 1.27)) hide)
-    )
-    (pin "1")
-  )
   (symbol (lib_id "Device:Crystal") (at 50.8 134.62 90) (unit 1)
     (in_bom yes) (on_board yes)
@@
     (pin "2")
   )
-  (symbol (lib_id "Power_Protection:SRV05-4") (at 63.5 58.42 0) (unit 1)
-    (in_bom yes) (on_board yes)
-    (property "Reference" "U5" (id 0) (at 72.39 63.5 0))
-    (property "Value" "SRV05-4" (id 1) (at 76.2 66.04 0))
-    (property "Footprint" "Package_TO_SOT_SMD:SOT-23-6" (id 2) (at 81.28 69.85 0)
-      (effects (font (size 1.27 1.27)) hide)
-    )
-    (property "Datasheet" "http://www.onsemi.com/pub/Collateral/SRV05-4-D.PDF" (id 3) (at 63.5 58.42 0)
-      (effects (font (size 1.27 1.27)) hide)
-    )
-    (pin "1")
-    (pin "2")
-    (pin "3")
-    (pin "4")
-    (pin "5")
-    (pin "6")
-  )
   (symbol (lib_id "Interface_Expansion:MCP23017_SP") (at 101.6 175.26 270) (unit 1)
     (in_bom yes) (on_board yes)
@@
       (reference "#PWR0134") (unit 1) (value "GND") (footprint "")
     )
-    (path "/3cb2dd4b-bfb2-4646-b3cb-bea68f5d9348"
-      (reference "#PWR0135") (unit 1) (value "VBUS") (footprint "")
-    )
     (path "/ea694357-f89b-4587-b390-485be1f22d2a"
       (reference "BZ1") (unit 1) (value "Buzzer") (footprint "Buzzer_Beeper:Buzzer_12x9.5RM7.6")
@@
       (reference "U4") (unit 1) (value "MCP23017_SP") (footprint "Package_DIP:DIP-28_W7.62mm")
     )
-    (path "/70f86704-7162-4d81-af00-44a1d7c0ec65"
-      (reference "U5") (unit 1) (value "SRV05-4") (footprint "Package_TO_SOT_SMD:SOT-23-6")
-    )
     (path "/3d1a9f74-df1a-46ac-a9df-74875a7a3850"
