File: Protopico/Protopico.kicad_pcb (KiCad board)
At the start: 4 copper layers, 86.1 x 50.8 mm, 60 parts, among them J1 Conn_01x03, J10 Conn_02x02_Odd_Even, J12 Conn_01x03, J13 USB_C_Receptacle, J2 Conn_01x01, J3 Conn_01x01, J4 Conn_01x01, J5 Conn_02x13_Odd_Even, J6 Conn_01x02, J7 Conn_02x02_Odd_Even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

Commit message: added images of the board
Parts:
- moved ? 189.1 mm to (232.2, 84.9)
- moved ? 164.6 mm to (224.0, 106.3)
- moved ? 57.3 mm to (157.6, 79.0)
Changed lines of the file:
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@@
   )
   (footprint "" (layer "F.Cu")
-    (at 60.96 165.1)
+    (at 232.18 84.89)
     (fp_text reference "" (at 0 0) (layer "F.SilkS")
       (effects (font (size 1.27 1.27) (thickness 0.15)))
@@
   )
   (footprint "" (layer "F.Cu")
-    (at 137.16 132.588)
+    (at 157.59 79.05)
     (fp_text reference "" (at 0 0) (layer "F.SilkS")
       (effects (font (size 1.27 1.27) (thickness 0.15)))
@@
   )
   (footprint "" (layer "F.Cu")
-    (at 59.69 116.84)
+    (at 223.99 106.26)
     (fp_text reference "" (at 0 0) (layer "F.SilkS")
       (effects (font (size 1.27 1.27) (thickness 0.15)))
@@
   (via (at 186.69 104.14) (size 1) (drill 0.4) (layers "F.Cu" "B.Cu") (free) (net 2))
   (via (at 181.102 79.756) (size 1) (drill 0.4) (layers "F.Cu" "B.Cu") (net 2))
-  (via (at 233.172 85.09) (size 1) (drill 0.4) (layers "F.Cu" "B.Cu") (free) (net 2))
+  (via (at 233.4 87.3) (size 1) (drill 0.4) (layers "F.Cu" "B.Cu") (free) (net 2))
   (via (at 195.072 100.584) (size 1) (drill 0.4) (layers "F.Cu" "B.Cu") (net 2))
   (via (at 189.992 81.788) (size 1) (drill 0.4) (layers "F.Cu" "B.Cu") (net 2))

Commit message: improved pcb and schematic
Parts:
- added C19: 100nF, Capacitor_SMD:C_1206_3216Metric_Pad1.33x1.80mm_HandSolder, F.Cu at (208.8, 105.2)
- added U5: SRV05-4, Package_TO_SOT_SMD:SOT-23-6, F.Cu at (140.7, 110.4)
- J13: value USB_C_Receptacle -> USB_C 2.0
- moved ? 12.5 mm to (235.8, 110.1)
- moved C7 2.16 mm to (178.4, 83.2), turned to 90 degrees
- moved R7 2.03 mm to (199.6, 104.1)
- moved R8 2.03 mm to (202.2, 104.1)
- moved U4 2.02 mm to (230.1, 108.0)
- moved C9 0.89 mm to (192.3, 85.7)
- moved ? 0.66 mm to (158.2, 79.1)
- moved SW1 0.57 mm to (230.6, 100.8)
- moved SW2 0.57 mm to (230.6, 104.6)
- moved C13 0.51 mm to (196.3, 88.6)
Routing:
- net +3V3: track 181.5 -> 241.2 mm, vias 0 -> 1
- net /GPA3: track 5.39 -> 28.3 mm
- net /GPA5: track 24.5 -> 8.77 mm
- net /GPA6: track 26.2 -> 13.8 mm
- net /GPA2: track 12.4 -> 23.1 mm
- net /GPIO2: track 149.7 -> 140.1 mm
- net /GPA0: track 20.6 -> 30.0 mm
- net /GPA4: track 15.8 -> 25.0 mm
- net /GPA7: track 25.9 -> 20.3 mm
- net /GPB6: track 24.8 -> 28.6 mm
- net /GPB5: track 25.3 -> 29.1 mm
- net /GPB1: track 25.7 -> 29.2 mm
- net /GPB2: track 25.9 -> 28.9 mm
- net /GPB4: track 25.9 -> 28.5 mm
- net /GPIO18: track 31.9 -> 34.5 mm
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Other:
- outline, holes or cut-outs redrawn
- board text added: "where?"

Commit message: improved pcb
Parts:
- removed U5: SRV05-4, Package_TO_SOT_SMD:SOT-23-6
Routing:
- net /GPIO23: track 39.1 -> 38.6 mm
- net Net-(R3-Pad2): track 3.21 -> 3.71 mm
Other:
- board text removed: "where?"

Commit message: added logo to pcb
Parts:
- added G***: LOGO, Symbol:DVB_SMALL, F.Cu at (173.2, 113.1)
